File: Breakout_Boards/Electrode_Breakout/Electrode_Breakout.kicad_sch (KiCad schematic)
At the start: 6 parts, among them J1 DB-9_Female, J2 DB-9_Female, J3 Conn_01x04_Pin, J4 Conn_01x04_Pin, J5 Conn_01x04_Pin, J7 Conn_01x03_Pin

Commit message: Push Electrode_Breakout to Git
Parts:
- removed J3, J4, J5: Conn_01x04_Pin, Connector_PinHeader_2.54mm:PinHeader_1x04_P2.54mm_Vertical, symbol Connector:Conn_01x04_Pin
- removed J7: Conn_01x03_Pin, Connector_PinHeader_2.54mm:PinHeader_1x03_P2.54mm_Vertical, symbol Connector:Conn_01x03_Pin
- added J3, J4: Conn_01x06, Connector_PinHeader_2.54mm:PinHeader_1x06_P2.54mm_Vertical, symbol Connector_Generic:Conn_01x06
- added J5, J6: Conn_01x03, Connector_PinHeader_2.54mm:PinHeader_1x03_P2.54mm_Vertical, symbol Connector_Generic:Conn_01x03
Connections:
- net +12V: now also J1.8, J2.7, J5.3 (Pin_3), J6.3 (Pin_3); no longer J1.2, J2.2
- net -12V: now also J1.7, J2.8, J5.2 (Pin_2), J6.2 (Pin_2); no longer J1.5, J2.5
- net ADC1: now also J1.9, J3.1 (Pin_1); no longer J1.1
- net ADC2: now also J1.5, J3.2 (Pin_2); no longer J1.9
- net ADC3: now also J4.5 (Pin_5)
- net ADC4: now also J2.6, J4.6 (Pin_6); no longer J2.9
- net CUR1: now also J1.1, J3.6 (Pin_6); no longer J1.3
- net CUR2: now also J1.2, J3.5 (Pin_5); no longer J1.7
- net CUR3: now also J2.2, J4.4 (Pin_4); no longer J2.3
- net CUR4: now also J2.3, J4.3 (Pin_3); no longer J2.7
- net GND: now also J2.9, J5.1 (Pin_1), J6.1 (Pin_1); no longer J2.6
- net SEL1: now also J1.3, J3.4 (Pin_4); no longer J1.4
- net SEL2: now also J1.4, J3.3 (Pin_3); no longer J1.8
- net SEL3: now also J4.2 (Pin_2)
- net SEL4: now also J2.5, J4.1 (Pin_1); no longer J2.8
